File: FPGA.sch (KiCad schematic (older format))
At the start: 87 parts, among them J1 Conn_02x05_Odd_Even, Q3 AO3400, Q4 AO3400, Q5 AO3400, U1 LFE5Ux-45F, U11 74LVC1G175, U2 LY68L6400SLIT, U3 LY68L6400SLIT, U4 W25Q128JVSIQ, U8 74LVC1G3157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

Commit message: Added measurements Labelled jtag signals
Parts:
- J1: symbol Connector_Generic:Conn_02x05_Odd_Even -> hadbadge2019-rescue:Conn_02x05_Odd_Even-Connector_Generic
- Q3, Q4, Q5: symbol jeroens_components:AO3400 -> hadbadge2019-rescue:AO3400-jeroens_components
- TP1, TP11, TP2, TP3, TP4, TP5, TP6, TP7: symbol Connector:TestPoint -> hadbadge2019-rescue:TestPoint-Connector
- U11: symbol 74xGxx:74LVC1G175 -> hadbadge2019-rescue:74LVC1G175-74xGxx
- U2, U3: symbol Lyontek_psram:LY68L6400SLIT -> hadbadge2019-rescue:LY68L6400SLIT-Lyontek_psram
- U4: symbol Memory_EEPROM:25LCxxx -> hadbadge2019-rescue:25LCxxx-Memory_EEPROM
- U8: symbol 74xGxx:74LVC1G3157 -> hadbadge2019-rescue:74LVC1G3157-74xGxx
- X1: symbol Oscillator:XO91 -> hadbadge2019-rescue:XO91-Oscillator
Connections:
- net labels added: TCK, TDI, TDO, TMS
Changed lines of the file:
@@
 Connection ~ 5600 9750
 $Comp
-L Connector:TestPoint TP11
+L hadbadge2019-rescue:TestPoint-Connector TP11
 U 1 1 5C610EE2
 P 6350 9650
@@
 VIO
 $Comp
-L Oscillator:XO91 X1
+L hadbadge2019-rescue:XO91-Oscillator X1
 U 1 1 5C790E80
 P 6100 7300
@@
 USB_VBUSDET
 $Comp
-L Lyontek_psram:LY68L6400SLIT U2
+L hadbadge2019-rescue:LY68L6400SLIT-Lyontek_psram U2
 U 1 1 5C736125
 P 10000 1750
@@
 $EndComp
 $Comp
-L Lyontek_psram:LY68L6400SLIT U3
+L hadbadge2019-rescue:LY68L6400SLIT-Lyontek_psram U3
 U 1 1 5C736206
 P 12350 1750
@@
 FLASH_MISO
 $Comp
-L Memory_EEPROM:25LCxxx U4
+L hadbadge2019-rescue:25LCxxx-Memory_EEPROM U4
 U 1 1 5C60DD62
 P 3600 9050
@@
 	7000 8050 7500 8050
 $Comp
-L Connector:TestPoint TP3
+L hadbadge2019-rescue:TestPoint-Connector TP3
 U 1 1 5D0D490B
 P 7150 3750
@@
 $EndComp
 $Comp
-L Connector:TestPoint TP4
+L hadbadge2019-rescue:TestPoint-Connector TP4
 U 1 1 5D0F5887
 P 7150 3950
@@
 $EndComp
 $Comp
-L Connector:TestPoint TP2
+L hadbadge2019-rescue:TestPoint-Connector TP2
 U 1 1 5D0FC9A7
 P 6950 2950
@@
 $EndComp
 $Comp
-L Connector:TestPoint TP1
+L hadbadge2019-rescue:TestPoint-Connector TP1
 U 1 1 5D101883
 P 7150 3350
@@
 $EndComp
 $Comp
-L 74xGxx:74LVC1G3157 U8
+L hadbadge2019-rescue:74LVC1G3157-74xGxx U8
 U 1 1 5D1561B3
 P 2100 7800
@@
 $EndComp
 $Comp
-L 74xGxx:74LVC1G175 U11
+L hadbadge2019-rescue:74LVC1G175-74xGxx U11
 U 1 1 5D157A6C
 P 1450 8100
@@
 Connection ~ 6750 1850
 $Comp
-L Connector_Generic:Conn_02x05_Odd_Even J1
+L hadbadge2019-rescue:Conn_02x05_Odd_Even-Connector_Generic J1
 U 1 1 5DA8142F
 P 6200 1550
@@
 DBGRX
 $Comp
-L Connector:TestPoint TP5
+L hadbadge2019-rescue:TestPoint-Connector TP5
 U 1 1 5DBBBFEA
 P 7150 3550
@@
 $EndComp
 $Comp
-L Connector:TestPoint TP6
+L hadbadge2019-rescue:TestPoint-Connector TP6
 U 1 1 5DBE8CB5
 P 9450 6050
@@
 Note: All LEDs indeed are RGB LEDs, but normally, \nonly CATA is powered so all LEDs will only light up \nin whatever color is connected to that. Good luck \ngetting full RGB!
 $Comp
-L jeroens_components:AO3400 Q3
+L hadbadge2019-rescue:AO3400-jeroens_components Q3
 U 1 1 5D8C68B4
 P 13400 9250
@@
 CATA
 $Comp
-L jeroens_components:AO3400 Q4
+L hadbadge2019-rescue:AO3400-jeroens_components Q4
 U 1 1 5D926D6D
 P 14550 9250
@@
 CATB
 $Comp
-L jeroens_components:AO3400 Q5
+L hadbadge2019-rescue:AO3400-jeroens_components Q5
 U 1 1 5D92F565
 P 15650 9250
@@
 $EndComp
 $Comp
-L Connector:TestPoint TP7
+L hadbadge2019-rescue:TestPoint-Connector TP7
 U 1 1 5D74ACE2
 P 1100 4750
@@
 Text GLabel 1100 6050 0    50   Input ~ 0
 GENIO_29
+Text Label 7100 1850 0    50   ~ 0
+TMS
+Text Label 7100 1750 0    50   ~ 0
+TDI
+Text Label 7100 1650 0    50   ~ 0
+TCK
+Text Label 6950 1550 0    50   ~ 0
+TDO
 $EndSCHEMATC
