File: hadbadge2019.kicad_pcb (KiCad board)
At the start: 4 copper layers, 88 x 140.5 mm, 204 parts, among them J1 Conn_02x05_Odd_Even, J10 Conn_01x02_Male, J11 NO STUFF, J12 NO STUFF, J2 USB_B_Micro, J3 NO STUFF, J4 HDMI_A_1.4, J5 FH26W-45S-0.3SHW(60), J6 Conn_02x20_Odd_Even, J7 Conn_02x03_Odd_Even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

Commit message: Added measurements Labelled jtag signals
Connections:
- net Net-(J1-Pad5) renamed /FPGA/TDI
- net Net-(J1-Pad6) renamed /FPGA/TDO
- net Net-(J1-Pad7) renamed /FPGA/TMS
- net Net-(J1-Pad8) renamed /FPGA/TCK
