File: outputs.sch (KiCad schematic (older format))
At the start: 68 parts, among them J10 Conn_01x02_Male, J11 NO STUFF, J12 NO STUFF, J2 USB_B_Micro, J3 NO STUFF, J4 HDMI_A_1.4, J5 FH26W-45S-0.3SHW(60), J6 Conn_02x20_Odd_Even, J7 Conn_02x03_Odd_Even, J8 Conn_02x03_Odd_Even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

Commit message: Added measurements Labelled jtag signals
Parts:
- J10, J9: symbol Connector:Conn_01x02_Male -> hadbadge2019-rescue:Conn_01x02_Male-Connector
- J11: symbol Connector_Generic:Conn_02x06_Odd_Even -> hadbadge2019-rescue:Conn_02x06_Odd_Even-Connector_Generic
- J12: symbol Connector:Conn_01x04_Female -> hadbadge2019-rescue:Conn_01x04_Female-Connector
- J2: symbol Connector:USB_B_Micro -> hadbadge2019-rescue:USB_B_Micro-Connector
- J3: symbol Connector_Generic:Conn_01x02 -> hadbadge2019-rescue:Conn_01x02-Connector_Generic
- J4: symbol Connector:HDMI_A_1.4 -> hadbadge2019-rescue:HDMI_A_1.4-Connector
- J5: symbol Connector_Generic_MountingPin:Conn_2Rows-45Pins_MountingPin -> hadbadge2019-rescue:Conn_2Rows-45Pins_MountingPin-Connector_Generic_MountingPin
- J6: symbol Connector_Generic:Conn_02x20_Odd_Even -> hadbadge2019-rescue:Conn_02x20_Odd_Even-Connector_Generic
- J7, J8: symbol Connector_Generic:Conn_02x03_Odd_Even -> hadbadge2019-rescue:Conn_02x03_Odd_Even-Connector_Generic
- Q1: symbol jeroens_components:AO3400 -> hadbadge2019-rescue:AO3400-jeroens_components
- SW1, SW2, SW3, SW4, SW5, SW6, SW7, SW8: symbol Switch:SW_Push -> hadbadge2019-rescue:SW_Push-Switch
- TP12, TP13, TP14, TP15: symbol Connector:TestPoint -> hadbadge2019-rescue:TestPoint-Connector
Changed lines of the file:
@@
 $EndDescr
 $Comp
-L Connector:USB_B_Micro J2
+L hadbadge2019-rescue:USB_B_Micro-Connector J2
 U 1 1 5C642886
 P 1250 1900
@@
 Connection ~ 1200 2300
 $Comp
-L Connector:HDMI_A_1.4 J4
+L hadbadge2019-rescue:HDMI_A_1.4-Connector J4
 U 1 1 5C642C42
 P 9850 2400
@@
 	8650 3100 8500 3100
 $Comp
-L Connector:TestPoint TP13
+L hadbadge2019-rescue:TestPoint-Connector TP13
 U 1 1 5C6809BB
 P 8500 2500
@@
 $EndComp
 $Comp
-L Connector:TestPoint TP14
+L hadbadge2019-rescue:TestPoint-Connector TP14
 U 1 1 5C680A80
 P 8500 2700
@@
 $EndComp
 $Comp
-L Connector:TestPoint TP15
+L hadbadge2019-rescue:TestPoint-Connector TP15
 U 1 1 5C680B1B
 P 8500 2800
@@
 $EndComp
 $Comp
-L Connector:TestPoint TP12
+L hadbadge2019-rescue:TestPoint-Connector TP12
 U 1 1 5C684690
 P 2300 2150
@@
 	3100 1200 3300 1200
 $Comp
-L Connector_Generic_MountingPin:Conn_2Rows-45Pins_MountingPin J5
+L hadbadge2019-rescue:Conn_2Rows-45Pins_MountingPin-Connector_Generic_MountingPin J5
 U 1 1 5C691D2E
 P 2450 4500
@@
 	2050 3700 2250 3700
 $Comp
-L jeroens_components:AO3400 Q1
+L hadbadge2019-rescue:AO3400-jeroens_components Q1
 U 1 1 5C6ADED4
 P 3850 3500
@@
 	2950 4000 2750 4000
 $Comp
-L Switch:SW_Push SW1
+L hadbadge2019-rescue:SW_Push-Switch SW1
 U 1 1 5C6B5595
 P 9350 4250
@@
 BTN_UP
 $Comp
-L Switch:SW_Push SW2
+L hadbadge2019-rescue:SW_Push-Switch SW2
 U 1 1 5C6BC3D6
 P 9350 4450
@@
 BTN_DOWN
 $Comp
-L Switch:SW_Push SW3
+L hadbadge2019-rescue:SW_Push-Switch SW3
 U 1 1 5C6C95C8
 P 9350 4650
@@
 BTN_LEFT
 $Comp
-L Switch:SW_Push SW4
+L hadbadge2019-rescue:SW_Push-Switch SW4
 U 1 1 5C6D0730
 P 9350 4850
@@
 BTN_RIGHT
 $Comp
-L Switch:SW_Push SW5
+L hadbadge2019-rescue:SW_Push-Switch SW5
 U 1 1 5C6D701C
 P 9350 5050
@@
 BTN_A
 $Comp
-L Switch:SW_Push SW6
+L hadbadge2019-rescue:SW_Push-Switch SW6
 U 1 1 5C6DD90C
 P 9350 5250
@@
 BTN_B
 $Comp
-L Switch:SW_Push SW7
+L hadbadge2019-rescue:SW_Push-Switch SW7
 U 1 1 5C6E41FE
 P 9350 5450
@@
 BTN_SELECT
 $Comp
-L Switch:SW_Push SW8
+L hadbadge2019-rescue:SW_Push-Switch SW8
 U 1 1 5C6EAAF2
 P 9350 5650
@@
 SNDOUT
 $Comp
-L Connector_Generic:Conn_01x02 J3
+L hadbadge2019-rescue:Conn_01x02-Connector_Generic J3
 U 1 1 5C78AF2B
 P 6650 1900
@@
 [38,39,40]=[im2,im1,im0]\n[0,0,0]=DBI type-B 18-bit
 $Comp
-L Connector_Generic:Conn_02x03_Odd_Even J7
+L hadbadge2019-rescue:Conn_02x03_Odd_Even-Connector_Generic J7
 U 1 1 5CEDF19E
 P 4000 6700
@@
 $EndComp
 $Comp
-L Connector_Generic:Conn_02x03_Odd_Even J8
+L hadbadge2019-rescue:Conn_02x03_Odd_Even-Connector_Generic J8
 U 1 1 5CEEDF6E
 P 5800 6700
@@
 $EndComp
 $Comp
-L Connector:Conn_01x02_Male J10
+L hadbadge2019-rescue:Conn_01x02_Male-Connector J10
 U 1 1 5CEEDF74
 P 5950 7100
@@
 $EndComp
 $Comp
-L Connector_Generic:Conn_02x20_Odd_Even J6
+L hadbadge2019-rescue:Conn_02x20_Odd_Even-Connector_Generic J6
 U 1 1 5D11B435
 P 5250 4900
@@
 SAO2_GPIO1
 $Comp
-L Connector:Conn_01x02_Male J9
+L hadbadge2019-rescue:Conn_01x02_Male-Connector J9
 U 1 1 5CEECB55
 P 4150 7050
@@
 $EndComp
 $Comp
-L Connector_Generic:Conn_02x06_Odd_Even J11
+L hadbadge2019-rescue:Conn_02x06_Odd_Even-Connector_Generic J11
 U 1 1 5D05A986
 P 7500 3900
@@
 $EndComp
 $Comp
-L Connector:Conn_01x04_Female J12
+L hadbadge2019-rescue:Conn_01x04_Female-Connector J12
 U 1 1 5D5BB0B7
 P 1800 1250
