File: power.sch (KiCad schematic (older format))
At the start: 47 parts, among them Q2 AO3401, SW9 SW_SPDT_shielded, U5 M3406, U6 XC6206P25, U7 XR1151, U9 XR1151

Commit message: Added measurements Labelled jtag signals
Parts:
- FID1, FID2, FID3, FID4, FID5, FID6: symbol Mechanical:Fiducial -> hadbadge2019-rescue:Fiducial-Mechanical
- H1: symbol Mechanical:MountingHole -> hadbadge2019-rescue:MountingHole-Mechanical
- Q2: symbol jeroens_components:AO3401 -> hadbadge2019-rescue:AO3401-jeroens_components
- SW9: symbol spdt_sh:SW_SPDT_shielded -> hadbadge2019-rescue:SW_SPDT_shielded-spdt_sh
- U5: symbol M3406:M3406 -> hadbadge2019-rescue:M3406-M3406
- U6: symbol xc6206:XC6206P25 -> hadbadge2019-rescue:XC6206P25-xc6206
Changed lines of the file:
@@
 $EndDescr
 $Comp
-L M3406:M3406 U5
+L hadbadge2019-rescue:M3406-M3406 U5
 U 1 1 5C5EF11E
 P 2900 2000
@@
 1V1
 $Comp
-L xc6206:XC6206P25 U6
+L hadbadge2019-rescue:XC6206P25-xc6206 U6
 U 1 1 5C5FCB13
 P 2900 3250
@@
 	6450 1950 6300 1950
 $Comp
-L spdt_sh:SW_SPDT_shielded SW9
+L hadbadge2019-rescue:SW_SPDT_shielded-spdt_sh SW9
 U 1 1 5CA14672
 P 6700 1950
@@
 $EndComp
 $Comp
-L jeroens_components:AO3401 Q2
+L hadbadge2019-rescue:AO3401-jeroens_components Q2
 U 1 1 5D6A27A7
 P 1350 2200
@@
 $EndComp
 $Comp
-L Mechanical:MountingHole H1
+L hadbadge2019-rescue:MountingHole-Mechanical H1
 U 1 1 5DBAD1B3
 P 6350 5100
@@
 $EndComp
 $Comp
-L Mechanical:Fiducial FID1
+L hadbadge2019-rescue:Fiducial-Mechanical FID1
 U 1 1 5D8D7810
 P 6400 5650
@@
 $EndComp
 $Comp
-L Mechanical:Fiducial FID2
+L hadbadge2019-rescue:Fiducial-Mechanical FID2
 U 1 1 5D8D81BD
 P 7000 5650
@@
 $EndComp
 $Comp
-L Mechanical:Fiducial FID3
+L hadbadge2019-rescue:Fiducial-Mechanical FID3
 U 1 1 5D8E19E9
 P 6400 6000
@@
 $EndComp
 $Comp
-L Mechanical:Fiducial FID4
+L hadbadge2019-rescue:Fiducial-Mechanical FID4
 U 1 1 5D8E19EF
 P 7000 6000
@@
 $EndComp
 $Comp
-L Mechanical:Fiducial FID5
+L hadbadge2019-rescue:Fiducial-Mechanical FID5
 U 1 1 5D8E7160
 P 6400 6350
@@
 $EndComp
 $Comp
-L Mechanical:Fiducial FID6
+L hadbadge2019-rescue:Fiducial-Mechanical FID6
 U 1 1 5D8E7166
 P 7000 6350
